File: hardware/main.sch (EAGLE design)
At the start: 9 parts, among them IC1 LD1117D33TR, Q1 BSS123

Commit message: Update schematics
Parts:
- R1: value 10k -> 39k
- R2: value 10k -> 68k
- R3: value 68k -> 10k
- R4: value 39k -> 10k
Changed lines of the file:
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@@
 <part name="P+2" library="supply1" deviceset="+5V" device=""/>
 <part name="+3V1" library="supply1" deviceset="+3V3" device=""/>
-<part name="R1" library="rcl" deviceset="R-EU_" device="M0805" value="10k"/>
-<part name="R2" library="rcl" deviceset="R-EU_" device="M0805" value="10k"/>
+<part name="R1" library="rcl" deviceset="R-EU_" device="M0805" value="39k"/>
+<part name="R2" library="rcl" deviceset="R-EU_" device="M0805" value="68k"/>
 <part name="GND3" library="supply1" deviceset="GND" device=""/>
 <part name="Q1" library="transistor-small-signal" deviceset="BSS123" device=""/>
-<part name="R3" library="rcl" deviceset="R-EU_" device="M0805" value="68k"/>
-<part name="R4" library="rcl" deviceset="R-EU_" device="M0805" value="39k"/>
+<part name="R3" library="rcl" deviceset="R-EU_" device="M0805" value="10k"/>
+<part name="R4" library="rcl" deviceset="R-EU_" device="M0805" value="10k"/>
 <part name="GND4" library="supply1" deviceset="GND" device=""/>
 <part name="GND5" library="supply1" deviceset="GND" device=""/>

Commit message: Update R4 value (thanks to @phoenix-de)
Parts:
- R4: value 10k -> 4.7k
Changed lines of the file:
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@@
 <part name="Q1" library="transistor-small-signal" deviceset="BSS123" device=""/>
 <part name="R3" library="rcl" deviceset="R-EU_" device="M0805" value="10k"/>
-<part name="R4" library="rcl" deviceset="R-EU_" device="M0805" value="10k"/>
+<part name="R4" library="rcl" deviceset="R-EU_" device="M0805" value="4.7k"/>
 <part name="GND4" library="supply1" deviceset="GND" device=""/>
 <part name="GND5" library="supply1" deviceset="GND" device=""/>
